Commit message: Add files via upload
Updated URDF model with motor parameters. Made multiple changes to the number of iterations and added a PD controller test file to determine the ideal kp and kd coefficients

File: 2DOFSinglelegmodel.urdf (robot description, URDF)
Before this commit: robot 2DOFSinglelegmodel, 5 links, 4 joints
Links:
- added link foot_link, mass 0.198271075333205; collision sphere radius=0.025; visual mesh filename=meshes/foot_link.STL
- link base_link: mass 1.05333227806636 -> 1.05333227963718; geometry collision mesh filename=meshes/base_link.STL; visual mesh filename=meshes/base_link.STL
- link hip_link: geometry collision mesh filename=meshes/hip_link.STL; visual mesh filename=meshes/hip_link.STL
- link knee_link: mass 0.333644599607618 -> 0.135373733148076
Joints:
- added joint foot_joint: type fixed, parent knee_link, child foot_link, origin xyz=0.075476 0.2007 0.082436 rpy=1.5708 0 -0.3597
- joint hip_joint: axis 0 1 0 -> -1 0 0; limit lower=-1.5708 upper=0 effort=0 velocity=0 -> lower=-1 upper=1.5708 effort=18.25 velocity=38.01327; origin xyz=0 -0.078825 0.060569 rpy=0 -0.066975 0 -> xyz=-0.0020938 -0.057691 0.094545 rpy=0 0 -1.5708
- joint knee_joint: limit lower=0 upper=2.0 effort=0 velocity=0 -> lower=0.5 upper=2.70 effort=18.25 velocity=38.01327; origin xyz=0.010925 -0.003674 0.14564 rpy=-1.5708 0 0 -> xyz=0.03081 0.0011539 0.14605 rpy=-1.5708 -0.066975 1.5708
- joint mount_joint: origin xyz=0 0 0 rpy=3.14159265 -1.5708 0 -> xyz=0 0 0 rpy=3.14159265 0 0
- joint pz_z: limit lower=-0.4 upper=0.3 effort=1000 velocity=20 -> lower=-0.40 upper=0.40 effort=1000 velocity=20; origin xyz=0 0 0.35 rpy=0 0 0 -> xyz=0 0 0.36 rpy=0 0 0
